File: board/Vaer.kicad_pcb (KiCad board)
At the start: 2 copper layers, 0 parts

Commit message: :construction: Start re-designing the PCB
Parts:
- added BT1: Battery_Cell, Battery:BatteryHolder_Keystone_1042_1x18650, F.Cu at (138.2, 80.1)
- added C1: 100nF, Capacitor_SMD:C_1206_3216Metric_Pad1.33x1.80mm_HandSolder, F.Cu at (123.6, 93.2)
- added C2: 100nF, Capacitor_SMD:C_1206_3216Metric_Pad1.33x1.80mm_HandSolder, F.Cu at (123.6, 96.5)
- added C3: 10uF, Capacitor_SMD:C_1206_3216Metric_Pad1.33x1.80mm_HandSolder, F.Cu at (123.6, 99.8)
- added C4: 10uF, Capacitor_SMD:C_1206_3216Metric_Pad1.33x1.80mm_HandSolder, F.Cu at (123.6, 103.2)
- added C5: 1uF, Capacitor_SMD:C_1206_3216Metric_Pad1.33x1.80mm_HandSolder, F.Cu at (123.6, 106.5)
- added C6: 1uF, Capacitor_SMD:C_1206_3216Metric_Pad1.33x1.80mm_HandSolder, F.Cu at (123.6, 109.9)
- added C7: 4.7uF, Capacitor_SMD:C_1206_3216Metric_Pad1.33x1.80mm_HandSolder, F.Cu at (123.6, 113.2)
- added D1: LED_BLUE_PWR, LED_SMD:LED_1206_3216Metric_Pad1.42x1.75mm_HandSolder, F.Cu at (154.8, 93.2)
- added D2: LED_YELLOW, LED_SMD:LED_1206_3216Metric_Pad1.42x1.75mm_HandSolder, F.Cu at (154.8, 96.6)
- added D3: LED_GREEN, LED_SMD:LED_1206_3216Metric_Pad1.42x1.75mm_HandSolder, F.Cu at (154.8, 100.0)
- added H1: MountingHole_Pad, MountingHole:MountingHole_2.5mm_Pad_Via, F.Cu at (140.4, 105.9)
- added H2: MountingHole_Pad, MountingHole:MountingHole_2.2mm_M2_Pad_Via, F.Cu at (148.7, 106.7)
- added H3: MountingHole_Pad, MountingHole:MountingHole_2.2mm_M2_Pad_Via, F.Cu at (148.7, 112.6)
- added H4: MountingHole_Pad, MountingHole:MountingHole_2.5mm_Pad_Via, F.Cu at (140.4, 112.4)
- added J1: Conn_01x03_Pin, Connector_PinHeader_1.00mm:PinHeader_1x03_P1.00mm_Vertical, F.Cu at (169.3, 93.0)
- added J2: Conn_01x03_Pin, Connector_PinHeader_1.00mm:PinHeader_1x03_P1.00mm_Vertical, F.Cu at (172.7, 93.0)
- added J3: Conn_01x04_Pin, Connector_PinHeader_1.00mm:PinHeader_1x04_P1.00mm_Vertical, F.Cu at (176.0, 93.0)
- added J4: GSB1C211110DS1HR, USB-C:AMPHENOL_GSB1C211110DS1HR, F.Cu at (132.4, 97.8)
- added R1: 10k, Resistor_SMD:R_1206_3216Metric_Pad1.30x1.75mm_HandSolder, F.Cu at (96.9, 93.1)
- added R2: 5k1, Resistor_SMD:R_1206_3216Metric_Pad1.30x1.75mm_HandSolder, F.Cu at (96.9, 96.4)
- added R3: 1k18, Resistor_SMD:R_1206_3216Metric_Pad1.30x1.75mm_HandSolder, F.Cu at (96.9, 99.7)
- added R4: 1k13, Resistor_SMD:R_1206_3216Metric_Pad1.30x1.75mm_HandSolder, F.Cu at (96.9, 103.0)
- added R5: 120, Resistor_SMD:R_1206_3216Metric_Pad1.30x1.75mm_HandSolder, F.Cu at (96.9, 106.3)
- added R6: 1k, Resistor_SMD:R_1206_3216Metric_Pad1.30x1.75mm_HandSolder, F.Cu at (96.9, 109.6)
- added R7: 1k, Resistor_SMD:R_1206_3216Metric_Pad1.30x1.75mm_HandSolder, F.Cu at (96.9, 112.9)
- added R8: 5k1, Resistor_SMD:R_1206_3216Metric_Pad1.30x1.75mm_HandSolder, F.Cu at (96.9, 116.2)
- added R9: 10k, Resistor_SMD:R_1206_3216Metric_Pad1.30x1.75mm_HandSolder, F.Cu at (96.9, 119.4)
- added SW_FLASH1: Flash mode, Button_Switch_THT:SW_PUSH_6mm, F.Cu at (128.6, 104.6)
- added SW_RESET1: Reset, Button_Switch_THT:SW_PUSH_6mm, F.Cu at (128.6, 113.2)
- added TP1: TestPoint, TestPoint:TestPoint_Pad_D1.0mm, F.Cu at (147.2, 93.0)
- added TP2: TestPoint, TestPoint:TestPoint_Pad_D1.0mm, F.Cu at (147.2, 96.0)
- added TP3: TestPoint, TestPoint:TestPoint_Pad_D1.0mm, F.Cu at (147.2, 99.1)
- added TP4: TestPoint, TestPoint:TestPoint_Pad_D1.0mm, F.Cu at (147.2, 102.2)
- added TP5: TestPoint, TestPoint:TestPoint_Pad_D1.0mm, F.Cu at (150.3, 93.0)
- added TP6: TestPoint, TestPoint:TestPoint_Pad_D1.0mm, F.Cu at (150.3, 96.0)
- added TP7: TestPoint, TestPoint:TestPoint_Pad_D1.0mm, F.Cu at (150.3, 99.1)
- added U1: BME280, Package_LGA:Bosch_LGA-8_2.5x2.5mm_P0.65mm_ClockwisePinNumbering, F.Cu at (160.0, 107.4)
- added U2: ESP32-S3-WROOM-1, Espressif:ESP32-S3-WROOM-1, F.Cu at (110.2, 108.1)
- added U3: NCP1117-3.3_SOT223, Package_TO_SOT_SMD:SOT-223-3_TabPin2, F.Cu at (162.7, 95.7)
- added U4: BQ24073RGT, Package_DFN_QFN:VQFN-16-1EP_3x3mm_P0.5mm_EP1.6x1.6mm, F.Cu at (160.4, 102.5)

Commit message: :construction: Group several components which should be cloth to each other
Parts:
- moved H2 158.7 mm to (279.8, 17.3)
- moved H1 152.2 mm to (16.9, 17.0)
- moved H4 147.4 mm to (16.8, 192.7)
- moved H3 138.4 mm to (278.3, 160.8)
- moved SW_FLASH1 130.8 mm to (17.2, 173.2)
- moved TP5 119.3 mm to (269.5, 96.5)
- moved TP6 119.3 mm to (269.5, 99.5)
- moved TP7 119.3 mm to (269.5, 102.5)
- moved TP1 119.3 mm to (266.4, 96.5)
- moved TP2 119.3 mm to (266.4, 99.5)
- moved TP3 119.3 mm to (266.4, 102.5)
- moved TP4 119.3 mm to (266.4, 105.6)
- moved SW_RESET1 113.2 mm to (32.5, 173.0)
- moved C5 111.9 mm to (28.7, 165.8)
- moved J4 108.3 mm to (25.1, 82.8), turned to -90 degrees
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